Commit message: change table collision

File: ycb_models_desc/urdf/pudding_box.urdf (robot description, URDF)
Before this commit: robot pudding_box, 2 links, 1 joints
Links:
- removed link world
Joints:
- removed joint fixed

File: ycb_models_desc/urdf/table.urdf (robot description, URDF)
Before this commit: robot box, 2 links, 1 joints
Links:
- link base_link: geometry collision box size=1.5 2.0 0.02; visual box size=1.5 2.0 0.02
