Commit message: corrected simulation

File: ycb_models_desc/urdf/mustard_bottle.urdf (robot description, URDF)
Before this commit: robot mustard_bottle, 1 links, 0 joints
Links:
- added link world
- link bottle_link: mass 1 -> 0.1; geometry collision mesh filename=package://ycb_models_desc/models/ycb/006_mustard_bottle/poi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; visual mesh filename=package://ycb_models_desc/models/ycb/006_mustard_bottle/poi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
Joints:
- added joint fixed: type fixed, parent world, child bottle_link

File: ycb_models_desc/urdf/power_drill.urdf (robot description, URDF)
Before this commit: robot power_drill, 1 links, 0 joints
Links:
- added link world
- link drill_link: mass 1 -> 0.1; geometry collision mesh filename=package://ycb_models_desc/models/ycb/035_power_drill/poisso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; visual mesh filename=package://ycb_models_desc/models/ycb/035_power_drill/poisso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
Joints:
- added joint fixed: type fixed, parent world, child drill_link

File: ycb_models_desc/urdf/pudding_box.urdf (robot description, URDF)
Before this commit: robot pudding_box, 1 links, 0 joints
Links:
- added link world
- link box_link: mass 1 -> 0.1; geometry collision mesh filename=package://ycb_models_desc/models/ycb/008_pudding_box/poisso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; visual mesh filename=package://ycb_models_desc/models/ycb/008_pudding_box/poisso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
Joints:
- added joint fixed: type fixed, parent world, child box_link

File: ycb_models_desc/urdf/table.urdf (robot description, URDF)
Before this commit: robot box, 2 links, 1 joints
Links:
- link base_link: geometry collision box size=2.0 3.0 0.02; visual box size=1.5 2.0 0.02

Commit message: Added Point Cloud normal and plane segmentation

File: ycb_models_desc/urdf/mustard_bottle.urdf (robot description, URDF)
Before this commit: robot mustard_bottle, 2 links, 1 joints
Links:
- link bottle_link: mass 0.1 -> 1
