Commit message: pudding box stable spawn

File: ycb_models_desc/urdf/table.urdf (robot description, URDF)
Before this commit: robot box, 2 links, 1 joints
Links:
- added link cylinder_link, mass 2; collision cylinder length=0.44 radius=0.10; visual cylinder length=0.44 radius=0.10
Joints:
- removed joint fixed
- added joint base_world_stand: type fixed, parent world, child base_link, origin xyz=0 0 0 rpy=0 0 0
- added joint table_stand: type fixed, parent base_link, child cylinder_link, origin xyz=-0.125 -0.2 -0.220 rpy=0 0 3.1416
